Commit message: drive_in_gazebo

File: description/robot.urdf.xacro (robot description, xacro)
@@ -2,3 +2,4 @@
 <robot xmlns:xacro="http://www.ros.org/wiki/xacro"  name="robot">
     <xacro:include filename="robot_core.xacro"/>
+    <xacro:include filename="gazebo_control.xacro"/>
 </robot>

File: description/robot_core.xacro (robot description, xacro)
@@ -1,11 +1,7 @@
 <?xml version="1.0"?>
-<robot xmlns:xacro="http://www.ros.org/wiki/xacro">
-    <!-- Include file chứa macro inertial -->
+<robot xmlns:xacro="http://www.ros.org/wiki/xacro" >
     <xacro:include filename="inertial_macros.xacro"/>
-    <!-- Khai báo hằng số -->
-    <xacro:property name="pi" value="3.141592653589793"/>
-    <!-- Định nghĩa màu -->
     <material name="white">
-        <color rgba="1 1 1 1"/>
+        <color rgba="1 1 1 1" />
     </material>
     <material name="orange">
@@ -18,7 +14,8 @@
         <color rgba="0 0 0 1"/>
     </material>
-    <!-- Link gốc -->
-    <link name="base_link"/>
-    <!-- Joint nối base_link với chassis -->
+    <!-- BASE LINK -->
+    <link name="base_link">
+    </link>
+    <!-- CHASSIS LINK -->
     <joint name="chassis_joint" type="fixed">
         <parent link="base_link"/>
@@ -26,5 +23,4 @@
         <origin xyz="-0.1 0 0"/>
     </joint>
-    <!-- Link chassis -->
     <link name="chassis">
         <visual>
@@ -45,12 +41,14 @@
         </xacro:inertial_box>
     </link>
-    <!-- Left wheel joint -->
+    <gazebo reference="chassis">
+        <material>Gazebo/White</material>
+    </gazebo>
+    <!-- LEFT WHEEL LINK -->
     <joint name="left_wheel_joint" type="continuous">
         <parent link="base_link"/>
         <child link="left_wheel"/>
-        <origin xyz="0 0.175 0" rpy="-${pi/2} 0 0"/>
+        <origin xyz="0 0.175 0" rpy="-${pi/2} 0 0" />
         <axis xyz="0 0 1"/>
     </joint>
-    <!-- Left wheel link -->
     <link name="left_wheel">
         <visual>
@@ -69,12 +67,14 @@
         </xacro:inertial_cylinder>
     </link>
-    <!-- Right wheel joint -->
+    <gazebo reference="left_wheel">
+        <material>Gazebo/Blue</material>
+    </gazebo>
+    <!-- RIGHT WHEEL LINK -->
     <joint name="right_wheel_joint" type="continuous">
         <parent link="base_link"/>
         <child link="right_wheel"/>
-        <origin xyz="0 -0.175 0" rpy="${pi/2} 0 0"/>
+        <origin xyz="0 -0.175 0" rpy="${pi/2} 0 0" />
         <axis xyz="0 0 -1"/>
     </joint>
-    <!-- Right wheel link -->
     <link name="right_wheel">
         <visual>
@@ -93,5 +93,8 @@
         </xacro:inertial_cylinder>
     </link>
-    <!-- Caster wheel joint -->
+    <gazebo reference="right_wheel">
+        <material>Gazebo/Blue</material>
+    </gazebo>
+    <!-- CASTER WHEEL LINK -->
     <joint name="caster_wheel_joint" type="fixed">
         <parent link="chassis"/>
@@ -99,5 +102,4 @@
         <origin xyz="0.24 0 0"/>
     </joint>
-    <!-- Caster wheel link -->
     <link name="caster_wheel">
         <visual>
@@ -116,3 +118,8 @@
         </xacro:inertial_sphere>
     </link>
+    <gazebo reference="caster_wheel">
+        <material>Gazebo/Black</material>
+        <mu1 value="0.001"/>
+        <mu2 value="0.001"/>
+    </gazebo>
 </robot>
