Commit message: lidar

File: description/gazebo_control.xacro (robot description, xacro)
@@ -1,4 +1,7 @@
 <?xml version="1.0"?>
 <robot xmlns:xacro="http://www.ros.org/wiki/xacro">
+    <!-- file nay su dung thu vien cho differential chi dieu khien duoc trong gazebo
+    Dung de test robot trong simulation, tat ca moi thu trong day chi hoat dong trong gazebo,
+    real khong su dung dc-->
     <gazebo>
         <plugin name="diff_drive" filename="libgazebo_ros_diff_drive.so">

File: description/robot.urdf.xacro (robot description, xacro)
@@ -2,4 +2,5 @@
 <robot xmlns:xacro="http://www.ros.org/wiki/xacro"  name="robot">
     <xacro:include filename="robot_core.xacro" />
-    <xacro:include filename="gazebo_control.xacro" />
+    <xacro:include filename="gazebo_control.xacro" /> <!-- File dkhien, pham vi trong gazebo-->
+    <xacro:include filename="lidar.xacro" />
 </robot>

File: description/robot_core.xacro (robot description, xacro)
@@ -13,4 +13,7 @@
     <material name="black">
         <color rgba="0 0 0 1"/>
+    </material>
+    <material name="red">
+        <color rgba="1 0 0 1"/>
     </material>
     <!-- BASE LINK -->
@@ -45,17 +48,22 @@
     </gazebo>
     <!-- LEFT WHEEL LINK -->
-    <joint name="left_wheel_joint" type="continuous">
-        <parent link="base_link"/>
-        <child link="left_wheel"/>
-        <origin xyz="0 0.175 0" rpy="-${pi/2} 0 0" />
-        <axis xyz="0 0 1"/>
+    <!--joint name: Quy định mối ghép. Quy định cách left wheel gắn vào Khungxe (base_link)-->
+    <joint name="left_wheel_joint" type="continuous"> <!--continuous khớp xoay không giới hạn-->
+        <parent link="base_link"/>  <!--Khung xe: đứng yên trong hệ quy chiếu -->
+        <child link="left_wheel"/>  <!--Left Wheel: đứng yên trong hệ quy chiếu -->
+        <origin xyz="0 0.175 0" rpy="-${pi/2} 0 0" /> <!--Bánh xe nằm lệch về phía trục Y (bên trái/0.175m)-->
+        <!--rpy="-${pi/2} 0 0": Mặc định hình trụ(cylinder) trong ROS đứng thẳng theo trục Z Để nằm ngang thành cái bánh xe,xoay nó -90 độ ($-\pi/2$) quanh trục X. -->
+        <axis xyz="0 0 1"/> <!--Trục quay cua wheel-->
     </joint>
+    <!--link name: Quy định hình dáng vật lý-->
     <link name="left_wheel">
+        <!--Thẻ hình ảnh hiển thị-->
         <visual>
-            <geometry>
-                <cylinder radius="0.05" length="0.04"/>
+            <geometry> <!--The hình học-->
+                <cylinder radius="0.05" length="0.04"/> <!--The hình trụ: r = 5cm, độ dày 4cm-->
             </geometry>
             <material name="blue"/>
         </visual>
+        <!--Thẻ va chạm vật lý, tinh toan trong gazebo-->
         <collision>
             <geometry>
@@ -63,9 +71,10 @@
             </geometry>
         </collision>
+        <!--Thẻ Quán tính-->
         <xacro:inertial_cylinder mass="0.1" length="0.04" radius="0.05">
             <origin xyz="0 0 0" rpy="0 0 0"/>
         </xacro:inertial_cylinder>
     </link>
-    <gazebo reference="left_wheel">
+    <gazebo reference="left_wheel">         <!--The hien thi trong gazebo-->
         <material>Gazebo/Orange</material>
     </gazebo>
