Commit message: all

File: description/camera.xacro (robot description, xacro)
@@ -5,5 +5,5 @@
         <parent link="chassis"/>
         <child link="camera_link"/>
-        <origin xyz="0.305 0 0.08" rpy="0 0 0"/>
+        <origin xyz="0.276 0 0.181" rpy="0 0 0"/>
     </joint>
     <!-- Hinh dang cua box camera -->
@@ -13,5 +13,12 @@
                 <box size="0.010 0.03 0.03"/>
             </geometry>
-            <material name="red"/>
+            <material name="black"/>
+        </visual>
+        <visual>
+            <origin xyz="0 0 -0.05"/>
+            <geometry>
+                <cylinder radius="0.002" length="0.1"/>
+            </geometry>
+            <material name="black"/>
         </visual>
     </link>
@@ -24,5 +31,5 @@
     <link name="camera_link_optical"></link>
     <gazebo reference="camera_link">
-        <material>Gazebo/Red</material>
+        <material>Gazebo/Black</material>
         <!--Plugin Camera hoat dong trong Gazebo-->
         <sensor name="camera" type="camera">
@@ -34,5 +41,5 @@
                 <image>
                     <format>R8G8B8</format>
-                    <width>640</width>  <!--Độ phân giải-->
+                    <width>640</width> <!--Độ phân giải-->
                     <height>480</height>
                 </image>

File: description/lidar.xacro (robot description, xacro)
@@ -4,5 +4,5 @@
         <parent link="chassis"/>
         <child link="laser_frame"/>
-        <origin xyz="0.1 0 0.175" rpy="0 0 0"/>
+        <origin xyz="0.122 0 0.212" rpy="0 0 0"/>
     </joint>
     <link name="laser_frame">
@@ -11,5 +11,12 @@
                 <cylinder radius="0.05" length="0.04"/>
             </geometry>
-            <material name="red"/>
+            <material name="black"/>
+        </visual>
+        <visual>
+            <origin xyz="0 0 -0.05"/>
+            <geometry>
+                <cylinder radius="0.01" length="0.1"/>
+            </geometry>
+            <material name="black"/>
         </visual>
         <collision>
@@ -23,6 +30,6 @@
     </link>
     <gazebo reference="laser_frame">
-        <material>Gazebo/Red</material>
-        <sensor name="laser" type="ray"> <!--Ray Tracing-->
+        <material>Gazebo/Black</material>
+        <sensor name="laser" type="ray">  <!--Ray Tracing-->
             <pose> 0 0 0 0 0 0 </pose>
             <visualize>false</visualize>
@@ -31,5 +38,5 @@
                 <scan>
                     <horizontal>
-                        <samples>360</samples>  <!-- 1 vòng quay nó lấy 360 điểm dữ liệu -->
+                        <samples>360</samples> <!-- 1 vòng quay nó lấy 360 điểm dữ liệu -->
                         <min_angle>-3.14</min_angle>
                         <max_angle>3.14</max_angle>
@@ -37,5 +44,5 @@
                 </scan>
                 <range>
-                    <min>0.1</min>
+                    <min>0.3</min>
                     <max>8</max> <!--Pham vi do dc max-->
                 </range>
@@ -44,5 +51,5 @@
             <plugin name="laser_controller" filename="libgazebo_ros_ray_sensor.so"> <!--Library simulate lidar in ROS-->
                 <ros>
-                    <argument>~/out:=scan</argument> <!--đổi tên topic, Mặc định plugin sẽ public ra topic tên dài -->
+                    <argument>~/out:=scan</argument> <!--đổi tên topic, Mặc định plugin sẽ public ra topic khac-->
                 </ros>
                 <output_type>sensor_msgs/LaserScan</output_type> <!--Publish ra array data -->

File: description/robot.urdf.xacro (robot description, xacro)
@@ -1,7 +1,12 @@
 <?xml version="1.0"?>
 <robot xmlns:xacro="http://www.ros.org/wiki/xacro"  name="robot">
+    <xacro:arg name="use_ros2_control" default="true"/>
     <xacro:include filename="robot_core.xacro" />
-    <!--<xacro:include filename="gazebo_control.xacro" /> -->  <!-- File dkhien, pham vi trong gazebo-->
-    <xacro:include filename="ros2_control.xacro" />
+    <xacro:if value="$(arg use_ros2_control)">
+        <xacro:include filename="ros2_control.xacro" />
+    </xacro:if>
+    <xacro:unless value="$(arg use_ros2_control)">
+        <xacro:include filename="gazebo_control.xacro" />
+    </xacro:unless>
     <xacro:include filename="lidar.xacro" />
     <xacro:include filename="camera.xacro" />

File: description/robot_core.xacro (robot description, xacro)
@@ -6,9 +6,9 @@
     <xacro:property name="chassis_height" value="0.138"/>
     <xacro:property name="chassis_mass" value="1.0"/>
-    <xacro:property name="wheel_radius" value="0.034"/>
+    <xacro:property name="wheel_radius" value="0.033"/>
     <xacro:property name="wheel_thickness" value="0.026"/>
     <xacro:property name="wheel_mass" value="0.05"/>
     <xacro:property name="wheel_offset_x" value="0.226"/>
-    <xacro:property name="wheel_offset_y" value="0.166"/>
+    <xacro:property name="wheel_offset_y" value="0.1485"/>
     <xacro:property name="wheel_offset_z" value="0.01"/>
     <xacro:property name="caster_wheel_radius" value="0.01"/>
@@ -46,5 +46,5 @@
                 <box size="${chassis_length} ${chassis_width} ${chassis_height}"/>
             </geometry>
-            <material name="orange"/>
+            <material name="white"/>
         </visual>
         <collision>
@@ -62,21 +62,17 @@
     </gazebo>
     <!-- LEFT WHEEL LINK -->
-    <!--joint name: Quy định mối ghép. Quy định cách left wheel gắn vào Khungxe (base_link)-->
-    <joint name="left_wheel_joint" type="continuous"> <!--continuous khớp xoay không giới hạn-->
-        <parent link="base_link"/>  <!--Khung xe: đứng yên trong hệ quy chiếu -->
-        <child link="left_wheel"/>  <!--Left Wheel: đứng yên trong hệ quy chiếu -->
-        <origin xyz="0 ${wheel_offset_y} 0" rpy="-${pi/2} 0 0" />   <!--Bánh xe nằm lệch về phía trục Y (bên trái/0.175m)-->
-        <axis xyz="0 0 1"/> <!--Trục quay cua wheel-->
+    <joint name="left_wheel_joint" type="continuous">
+        <parent link="base_link"/>
+        <child link="left_wheel"/>
+        <origin xyz="0 ${wheel_offset_y} 0" rpy="-${pi/2} 0 0" />
+        <axis xyz="0 0 1"/>
     </joint>
-    <!--link name: Quy định hình dáng vật lý-->
     <link name="left_wheel">
-        <!--Thẻ hình ảnh hiển thị-->
         <visual>
-            <geometry>  <!--The hình học-->
-                <cylinder radius="${wheel_radius}" length="${wheel_thickness}"/> <!--The hình trụ: r = 5cm, độ dày 4cm-->
+            <geometry>
+                <cylinder radius="${wheel_radius}" length="${wheel_thickness}"/>
             </geometry>
             <material name="blue"/>
         </visual>
-        <!--Thẻ va chạm vật lý, tinh toan trong gazebo-->
         <collision>
             <geometry>
@@ -84,10 +80,8 @@
             </geometry>
         </collision>
-        <!--Thẻ Quán tính-->
         <xacro:inertial_cylinder mass="${wheel_mass}" length="${wheel_thickness}" radius="${wheel_radius}">
             <origin xyz="0 0 0" rpy="0 0 0"/>
         </xacro:inertial_cylinder>
     </link>
-    <!--The hien thi trong gazebo-->
     <gazebo reference="left_wheel">
         <material>Gazebo/Blue</material>
@@ -117,5 +111,5 @@
     </link>
     <gazebo reference="right_wheel">
-        <material>Gazebo/Orange</material>
+        <material>Gazebo/Blue</material>
     </gazebo>
     <!-- CASTER WHEEL LINK -->

Commit message: fix_urdf

File: description/camera.xacro (robot description, xacro)
@@ -5,5 +5,5 @@
         <parent link="chassis"/>
         <child link="camera_link"/>
-        <origin xyz="0.276 0 0.181" rpy="0 0 0"/>
+        <origin xyz="0.150 0 0.150" rpy="0 0 0"/>
     </joint>
     <!-- Hinh dang cua box camera -->

File: description/lidar.xacro (robot description, xacro)
@@ -4,10 +4,10 @@
         <parent link="chassis"/>
         <child link="laser_frame"/>
-        <origin xyz="0.122 0 0.212" rpy="0 0 0"/>
+        <origin xyz="0.050 0 0.150" rpy="0 0 0"/>
     </joint>
     <link name="laser_frame">
         <visual>
             <geometry>
-                <cylinder radius="0.05" length="0.04"/>
+                <cylinder radius="0.030" length="0.022"/>
             </geometry>
             <material name="black"/>

File: description/robot_core.xacro (robot description, xacro)
@@ -2,13 +2,13 @@
 <robot xmlns:xacro="http://www.ros.org/wiki/xacro" >
     <xacro:include filename="inertial_macros.xacro"/>
-    <xacro:property name="chassis_length" value="0.335"/>
-    <xacro:property name="chassis_width" value="0.265"/>
-    <xacro:property name="chassis_height" value="0.138"/>
+    <xacro:property name="chassis_length" value="0.18"/>  <!--Chieu Dai -->
+    <xacro:property name="chassis_width" value="0.10"/>    <!--Chieu Rong -->
+    <xacro:property name="chassis_height" value="0.13"/>   <!--Chieu Cao -->
     <xacro:property name="chassis_mass" value="1.0"/>
-    <xacro:property name="wheel_radius" value="0.033"/>
-    <xacro:property name="wheel_thickness" value="0.026"/>
+    <xacro:property name="wheel_radius" value="0.033"/>     <!--Ban Kinh Banh Xe -->
+    <xacro:property name="wheel_thickness" value="0.026"/>  <!--Do day cua banh xe -->
     <xacro:property name="wheel_mass" value="0.05"/>
-    <xacro:property name="wheel_offset_x" value="0.226"/>
-    <xacro:property name="wheel_offset_y" value="0.1485"/>
+    <xacro:property name="wheel_offset_x" value="0.15"/>
+    <xacro:property name="wheel_offset_y" value="0.07"/>  <!--Nua K/cach 2 banh -->
     <xacro:property name="wheel_offset_z" value="0.01"/>
     <xacro:property name="caster_wheel_radius" value="0.01"/>
